File: stm32_lqfp48_breakout/stm32_lqfp48_breakout.kicad_sch (KiCad schematic)
At the start: 11 parts, among them J1 Conn_01x22, J2 Conn_01x22, U1 STM32L452CETx

Commit message: Finalized breakout for L-series
Parts:
- J1, J2: footprint (none) -> Connector_PinHeader_2.54mm:PinHeader_1x22_P2.54mm_Vertical
Connections:
- net VDD: now also J1.1 (Pin_1)
- net VDDA: now also J1.9 (Pin_9)
- net VDDUSB: now also J2.12 (Pin_12)
- net VSS: now also J2.1 (Pin_1)
- net VSSA: now also J1.8 (Pin_8)
- net PA0: now reaches J1.10 (Pin_10)
- net PA0: now also U1.10 (PA0)
- net PA1: now reaches J1.11 (Pin_11)
- net PA1: now also U1.11 (PA1)
- net PA2: now reaches J1.12 (Pin_12)
- net PA2: now also U1.12 (PA2)
- net PA3: now reaches J1.13 (Pin_13)
- net PA3: now also U1.13 (PA3)
- net PA4: now reaches J1.14 (Pin_14)
- net PA4: now also U1.14 (PA4)
- net PA5: now reaches J1.15 (Pin_15)
- net PA5: now also U1.15 (PA5)
- net PA6: now reaches J1.16 (Pin_16)
- net PA6: now also U1.16 (PA6)
- net PA7: now reaches J1.17 (Pin_17)
- net PA7: now also U1.17 (PA7)
- net PB0: now reaches J1.18 (Pin_18)
- net PB0: now also U1.18 (PB0)
- net PB1: now reaches J1.19 (Pin_19)
- net PB1: now also U1.19 (PB1)
- net PC13: now reaches J1.2 (Pin_2)
- net PC13: now also U1.2 (PC13)
- net PB2: now reaches J1.20 (Pin_20)
- net PB2: now also U1.20 (PB2)
- net PB10: now reaches J1.21 (Pin_21)
- net PB10: now also U1.21 (PB10)
- net PB11: now reaches J1.22 (Pin_22)
- net PB11: now also U1.22 (PB11)
- net PC14: now reaches J1.3 (Pin_3)
- net PC14: now also U1.3 (PC14)
- net PC15: now reaches J1.4 (Pin_4)
- net PC15: now also U1.4 (PC15)
- net PH0: now reaches J1.5 (Pin_5)
- net PH0: now also U1.5 (PH0)
- net PH1: now reaches J1.6 (Pin_6)
- net PH1: now also U1.6 (PH1)
- net NRST: now reaches J1.7 (Pin_7)
- net NRST: now also U1.7 (NRST)
- net PB12: now reaches U1.25 (PB12)
- net PB12: now also J2.22 (Pin_22)
- net PB13: now reaches U1.26 (PB13)
- net PB13: now also J2.21 (Pin_21)
- net PB14: now reaches U1.27 (PB14)
- net PB14: now also J2.20 (Pin_20)
- net PB15: now reaches U1.28 (PB15)
- net PB15: now also J2.19 (Pin_19)
- net PA8: now reaches U1.29 (PA8)
- net PA8: now also J2.18 (Pin_18)
- net PA9: now reaches U1.30 (PA9)
- net PA9: now also J2.17 (Pin_17)
- net PA10: now reaches U1.31 (PA10)
- net PA10: now also J2.16 (Pin_16)
- net PA11: now reaches U1.32 (PA11)
- net PA11: now also J2.15 (Pin_15)
- net PA12: now reaches U1.33 (PA12)
- net PA12: now also J2.14 (Pin_14)
- net PA13: now reaches U1.34 (PA13)
- net PA13: now also J2.13 (Pin_13)
- net PA14: now reaches U1.37 (PA14)
- net PA14: now also J2.11 (Pin_11)
- net PA15: now reaches U1.38 (PA15)
- net PA15: now also J2.10 (Pin_10)
- net PB3: now reaches U1.39 (PB3)
- net PB3: now also J2.9 (Pin_9)
- net PB4: now reaches U1.40 (PB4)
- net PB4: now also J2.8 (Pin_8)
- net PB5: now reaches U1.41 (PB5)
- net PB5: now also J2.7 (Pin_7)
- net PB6: now reaches U1.42 (PB6)
- net PB6: now also J2.6 (Pin_6)
- net PB7: now reaches U1.43 (PB7)
- net PB7: now also J2.5 (Pin_5)
- net PH3: now reaches U1.44 (PH3)
- net PH3: now also J2.4 (Pin_4)
- net PB8: now reaches U1.45 (PB8)
- net PB8: now also J2.3 (Pin_3)
- net PB9: now reaches U1.46 (PB9)
- net PB9: now also J2.2 (Pin_2)
