File: stm32g0x1_lqfp48_breakout/stm32g0x1_lqfp48_breakout.kicad_pcb (KiCad board)
At the start: 2 copper layers, 18.5 x 62 mm, 10 parts, among them J1 Conn_01x24, J2 Conn_01x24, J3 Conn_02x07_Odd_Even, SW1 SW_Push, U1 STM32G071CBTx

Commit message: Finalized G0x1 breakouts
Other:
- board text added: "3V3"
- board text added: "GND"
- board text removed: "VDD"
- board text removed: "VSS"
Changed lines of the file:
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@@
 		)
 		(property "Value" "Conn_02x07_Odd_Even"
-			(at 0 5.145 360)
+			(at 0 5.145 0)
 			(layer "F.Fab")
 			(effects
@@
 		)
 	)
-	(gr_text "VSS"
-		(at 152.75 71.5 0)
+	(gr_text "GND"
+		(at 152.5 71.5 0)
 		(layer "F.SilkS")
 		(effects
@@
 		)
 	)
-	(gr_text "VDD"
-		(at 144.25 71.5 0)
+	(gr_text "3V3"
+		(at 144 71.5 0)
 		(layer "F.SilkS")
 		(effects
