File: stm32g0x1_ufqfpn32_breakout/stm32g0x1_ufqfpn32_breakout.kicad_sch (KiCad schematic)
At the start: 8 parts, among them J1 Conn_01x16, J2 Conn_01x16, J3 Conn_02x07_Odd_Even, SW1 SW_Push, U1 STM32G071K8Tx

Commit message: Finalized G0x1 breakouts
Parts:
- removed U1: STM32G071K8Tx, Package_QFP:LQFP-32_7x7mm_P0.8mm, symbol MCU_ST_STM32G0:STM32G071K8Tx
- added U1: STM32G071KBUx, Package_DFN_QFN:QFN-32-1EP_5x5mm_P0.5mm_EP3.45x3.45mm, symbol MCU_ST_STM32G0:STM32G071KBUx
Connections:
- net NRST: now also J1.2 (Pin_2), U1.6 (PF2); no longer J1.5 (Pin_5)
- net PA0: now also J1.3 (Pin_3), U1.7 (PA0); no longer J1.6 (Pin_6)
- net PA1: now also J1.4 (Pin_4), U1.8 (PA1); no longer J1.7 (Pin_7)
- net PA10: now also J2.16 (Pin_16), U1.21 (PA10/UCPD1_DBCC2); no longer J2.13 (Pin_13)
- net PA11: now also J2.15 (Pin_15), U1.22 (PA11/PA9); no longer J2.12 (Pin_12)
- net PA12: now also J2.14 (Pin_14), U1.23 (PA12/PA10); no longer J2.11 (Pin_11)
- net PA13: now also J2.13 (Pin_13), U1.24 (PA13); no longer J2.10 (Pin_10)
- net PA14: now also J2.12 (Pin_12), U1.25 (PA14); no longer J2.9 (Pin_9)
- net PA15: now also J2.11 (Pin_11), U1.26 (PA15); no longer J2.8 (Pin_8)
- net PA2: now also J1.5 (Pin_5), U1.9 (PA2); no longer J1.8 (Pin_8)
- net PA3: now also J1.6 (Pin_6), U1.10 (PA3); no longer J1.9 (Pin_9)
- net PA4: now also J1.7 (Pin_7), U1.11 (PA4); no longer J1.10 (Pin_10)
- net PA5: now also J1.8 (Pin_8), U1.12 (PA5); no longer J1.11 (Pin_11)
- net PA6: now also J1.9 (Pin_9), U1.13 (PA6); no longer J1.12 (Pin_12)
- net PA7: now also J1.10 (Pin_10), U1.14 (PA7); no longer J1.13 (Pin_13)
- net PA8: now also J1.14 (Pin_14), U1.18 (PA8); no longer J2.16 (Pin_16)
- net PA9: now also J1.15 (Pin_15), U1.19 (PA9/UCPD1_DBCC1); no longer J2.15 (Pin_15)
- net PB0: now also J1.11 (Pin_11), U1.15 (PB0); no longer J1.14 (Pin_14)
- net PB1: now also J1.12 (Pin_12), U1.16 (PB1); no longer J1.15 (Pin_15)
- net PB2: now also J1.13 (Pin_13), U1.17 (PB2); no longer J1.16 (Pin_16)
- net PB3: now also J2.10 (Pin_10), U1.27 (PB3); no longer J2.7 (Pin_7)
- net PB4: now also J2.9 (Pin_9), U1.28 (PB4); no longer J2.6 (Pin_6)
- net PB5: now also J2.8 (Pin_8), U1.29 (PB5); no longer J2.5 (Pin_5)
- net PB6: now also J2.7 (Pin_7), U1.30 (PB6); no longer J2.4 (Pin_4)
- net PB7: now also J2.6 (Pin_6), U1.31 (PB7); no longer J2.3 (Pin_3)
- net PB8: now also J2.5 (Pin_5), U1.32 (PB8); no longer J2.2 (Pin_2)
- net PB9: now also J2.4 (Pin_4), U1.1 (PB9); no longer J1.2 (Pin_2)
- net PC14: now also J2.3 (Pin_3), U1.2 (PC14); no longer J1.3 (Pin_3)
- net PC15: now also J2.2 (Pin_2), U1.3 (PC15); no longer J1.4 (Pin_4)
- net PC6: now also J1.16 (Pin_16), U1.20 (PC6); no longer J2.14 (Pin_14)
- net VDD: now also J2.1 (Pin_1), U1.4 (VDD); no longer J1.1 (Pin_1)
- net VSS: now also J1.1 (Pin_1), U1.33 (VSS), U1.5 (VSS); no longer J2.1 (Pin_1)
