File: USB_Battery_breakout/USB_Battery_breakout.kicad_pcb (KiCad board)
At the start: 2 copper layers, 20.5 x 36.5 mm, 33 parts, among them J1 USB_C_Receptacle_USB2.0_16P, J2 Conn_01x03, J3 Conn_01x06, J4 Conn_01x06, SW1 SW_Push, U1 BQ24259RGER, U2 TPS7A0533PDBV

Commit message: Make PG LED green, STAT red
STAT is usually an error, PG is normal operation.
Added JLCPCB part numbers for more components.
Parts:
- D2: value Green -> Red
- D3: value Red -> Green
- R2: value 220 -> 470
- R3: value 470 -> 220
Changed lines of the file:
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@@
 		(tags "connector JST PH horizontal")
 		(property "Reference" "J2"
-			(at 4.25 -4.5 360)
+			(at 4.25 -4.5 0)
 			(layer "F.SilkS")
 			(effects
@@
 		(tags "resistor")
 		(property "Reference" "R11"
-			(at 0 -1.17 360)
+			(at 0 -1.17 0)
 			(layer "F.SilkS")
 			(effects
@@
 		)
 		(property "Value" "200k"
-			(at 0 1.17 360)
+			(at 0 1.17 0)
 			(layer "F.Fab")
 			(effects
@@
 		)
 		(fp_text user "${REFERENCE}"
-			(at 0 0 360)
+			(at 0 0 0)
 			(layer "F.Fab")
 			(effects
@@
 			)
 		)
-		(property "Value" "Red"
+		(property "Value" "Green"
 			(at 0 1.43 0)
 			(layer "F.Fab")
@@
 			)
 		)
-		(property "JLCPCB" "C2286"
+		(property "JLCPCB" "C72043"
 			(at 0 0 0)
 			(unlocked yes)
@@
 		(tags "resistor")
 		(property "Reference" "R3"
-			(at -2 0 360)
+			(at -2 0 0)
 			(layer "F.SilkS")
 			(effects
@@
 			)
 		)
-		(property "Value" "470"
-			(at 0 1.17 360)
+		(property "Value" "220"
+			(at 0 1.17 0)
 			(layer "F.Fab")
 			(effects
@@
 			)
 		)
-		(property "JLCPCB" "C25117"
+		(property "JLCPCB" "C25091"
 			(at 0 0 180)
 			(unlocked yes)
@@
 		)
 		(fp_text user "${REFERENCE}"
-			(at 0 0 360)
+			(at 0 0 0)
 			(layer "F.Fab")
 			(effects
@@
 		(tags "SOT TO_SOT_SMD")
 		(property "Reference" "U2"
-			(at 0 2.5 360)
+			(at 0 2.5 0)
 			(layer "F.SilkS")
 			(effects
@@
 		)
 		(property "Value" "TPS7A0533PDBV"
-			(at 0 2.4 360)
+			(at 0 2.4 0)
 			(layer "F.Fab")
 			(effects
@@
 		)
 		(property "Footprint" "Package_TO_SOT_SMD:SOT-23-5"
-			(at 0 0 360)
+			(at 0 0 0)
 			(layer "F.Fab")
 			(hide yes)
@@
 		)
 		(property "Datasheet" "https://www.ti.com/lit/ds/symlink/tps7a05.pdf"
-			(at 0 0 360)
+			(at 0 0 0)
 			(layer "F.Fab")
 			(hide yes)
@@
 		)
 		(property "Description" "200-mA Ultra-Low-Iq LDO, 3.3V, SOT-23-5"
-			(at 0 0 360)
+			(at 0 0 0)
 			(layer "F.Fab")
 			(hide yes)
@@
 		)
 		(fp_text user "${REFERENCE}"
-			(at 0 0 360)
+			(at 0 0 0)
 			(layer "F.Fab")
 			(effects
@@
 		(tags "capacitor")
 		(property "Reference" "C11"
-			(at 0 1.25 360)
+			(at 0 1.25 0)
 			(layer "F.SilkS")
 			(effects
@@
 		)
 		(property "Value" "1u"
-			(at 0 1.16 360)
+			(at 0 1.16 0)
 			(layer "F.Fab")
 			(effects
@@
 		)
 		(fp_text user "${REFERENCE}"
-			(at 0 0 360)
+			(at 0 0 0)
 			(layer "F.Fab")
 			(effects
@@
 		(tags "resistor")
 		(property "Reference" "R2"
-			(at -1.99 0 360)
+			(at -1.99 0 0)
 			(layer "F.SilkS")
 			(effects
@@
 			)
 		)
-		(property "Value" "220"
-			(at 0 1.17 360)
+		(property "Value" "470"
+			(at 0 1.17 0)
 			(layer "F.Fab")
 			(effects
@@
 			)
 		)
-		(property "JLCPCB" "C25091"
+		(property "JLCPCB" "C25117"
 			(at 0 0 180)
 			(unlocked yes)
@@
 		)
 		(fp_text user "${REFERENCE}"
-			(at 0 0 360)
+			(at 0 0 0)
 			(layer "F.Fab")
 			(effects
@@
 		(tags "capacitor")
 		(property "Reference" "C6"
-			(at 0 1.25 360)
+			(at 0 1.25 0)
 			(layer "F.SilkS")
 			(effects
@@
 		)
 		(property "Value" "1u"
-			(at 0 1.16 360)
+			(at 0 1.16 0)
 			(layer "F.Fab")
 			(effects
@@
 		)
 		(fp_text user "${REFERENCE}"
-			(at 0 0 360)
+			(at 0 0 0)
 			(layer "F.Fab")
 			(effects
@@
 			)
 		)
+		(property "JLCPCB" "C3025063"
+			(at 0 0 0)
+			(unlocked yes)
+			(layer "F.Fab")
+			(hide yes)
+			(effects
+				(font
+					(size 1 1)
+					(thickness 0.15)
+				)
+			)
+		)
 		(property ki_fp_filters "USB*C*Receptacle*")
 		(sheetname "Root")
@@
 		)
 		(property "Value" "SW_Push"
-			(at 0 2.6 360)
+			(at 0 2.6 0)
 			(layer "F.Fab")
 			(effects
@@
 		)
 		(fp_text user "${REFERENCE}"
-			(at 0 0 360)
+			(at 0 0 0)
 			(layer "F.Fab")
 			(effects
@@
 			)
 		)
-		(property "Value" "Green"
+		(property "Value" "Red"
 			(at 0 1.43 0)
 			(layer "F.Fab")
@@
 			)
 		)
-		(property "JLCPCB" "C72043"
+		(property "JLCPCB" "C2286"
 			(at 0 0 0)
 			(unlocked yes)
@@
 			)
 		)
+		(property "JLCPCB" "C161082"
+			(at 0 0 0)
+			(unlocked yes)
+			(layer "F.Fab")
+			(hide yes)
+			(effects
+				(font
+					(size 1 1)
+					(thickness 0.15)
+				)
+			)
+		)
 		(property ki_fp_filters "Choke_* *Coil* Inductor_* L_*")
 		(sheetname "Root")
@@
 		(tags "resistor")
 		(property "Reference" "R7"
-			(at 0 -1.17 360)
+			(at 0 -1.17 0)
 			(layer "F.SilkS")
 			(effects
@@
 		)
 		(property "Value" "240"
-			(at 0 1.17 360)
+			(at 0 1.17 0)
 			(layer "F.Fab")
 			(effects
@@
 		)
 		(fp_text user "${REFERENCE}"
-			(at 0 0 360)
+			(at 0 0 0)
 			(layer "F.Fab")
 			(effects
@@
 			)
 		)
-		(property "JLCPCB" ""
+		(property "JLCPCB" "C5142571"
 			(at 0 0 90)
 			(unlocked yes)
@@
 		(tags "capacitor")
 		(property "Reference" "C7"
-			(at 0 -1.25 360)
+			(at 0 -1.25 0)
 			(layer "F.SilkS")
 			(effects
@@
 		)
 		(property "Value" "1u"
-			(at 0 1.16 360)
+			(at 0 1.16 0)
 			(layer "F.Fab")
 			(effects
@@
 		)
 		(fp_text user "${REFERENCE}"
-			(at 0 0 360)
+			(at 0 0 0)
 			(layer "F.Fab")
 			(effects
