File: bigger_red_button/bigger_red_button.kicad_pcb (KiCad board)
At the start: 2 copper layers, 25.2 x 31.2 mm, 18 parts, among them J1 Conn_02x05_Odd_Even, J2 USB_C_Receptacle_USB2.0_16P, J3 Conn_02x01, J4 Conn_02x01, Q1 AO3400A, U1 USBLC6-2SC6, U2 TPS7A0533PDBV, U3 STM32G0B1KBTx

Commit message: Reroute PCB
Parts:
- removed J3, J4: Conn_02x01, Connector_PinHeader_2.54mm:PinHeader_1x02_P2.54mm_Vertical
- removed Q1: AO3400A, Package_TO_SOT_SMD:SOT-23
- added C5: 10u, Capacitor_SMD:C_0402_1005Metric, F.Cu at (165.1, 145.7)
- added C6: 10u, Capacitor_SMD:C_0402_1005Metric, F.Cu at (165.1, 143.7)
- added JP1: Jumper_2_Open, Connector_PinHeader_2.54mm:PinHeader_1x02_P2.54mm_Vertical, F.Cu at (156.0, 123.0)
- added JP2: Jumper_2_Open, Connector_PinHeader_2.54mm:PinHeader_1x02_P2.54mm_Vertical, F.Cu at (163.3, 123.0)
- added L1: 4u7, Inductor_SMD:L_1008_2520Metric, F.Cu at (165.6, 141.2)
- added R3: 100m, Resistor_SMD:R_1206_3216Metric, F.Cu at (172.0, 147.0)
- added U4: PAM2804, Package_TO_SOT_SMD:TSOT-23-5, F.Cu at (167.6, 145.4)
- BUT1: value SW_Push -> External Button
- LED1: value LED -> External LED
- U3: value STM32G0B1KBTx -> STM32C071FBPx; footprint Package_QFP:LQFP-32_7x7mm_P0.8mm -> Package_SO:TSSOP-20_4.4x6.5mm_P0.65mm
- moved LED1 24.4 mm to (172.0, 143.8), turned to 180 degrees
- moved U2 12.9 mm to (157.1, 133.9), turned to 0 degrees
- moved C1 12.5 mm to (154.5, 133.0), turned to 90 degrees
- moved J2 12.1 mm to (170.0, 124.5), turned to -90 degrees
- moved C2 10.6 mm to (160.1, 133.4), turned to -90 degrees
- moved C4 10.1 mm to (164.2, 133.1), turned to 90 degrees
- moved U3 9.64 mm to (169.6, 133.6), turned to 0 degrees
- moved C3 9.56 mm to (165.2, 133.1), turned to 90 degrees
- moved R2 6.75 mm to (163.0, 147.5)
- moved BUT1 6.27 mm to (156.0, 128.5), turned to -90 degrees
- moved R4 6.18 mm to (159.0, 128.5), turned to -90 degrees
- moved J1 5.25 mm to (156.8, 146.0)
- moved U1 5.25 mm to (156.8, 138.4)
- moved C7 5.06 mm to (160.0, 128.5), turned to 90 degrees
- moved R1 4.60 mm to (152.5, 140.0), turned to 180 degrees
- renumbered C5 to C1, C4 to C2, C2 to C3, C3 to C4, C1 to C7, J2 to J1, J1 to J2, R2 to R1, R3 to R2, R1 to R4
Connections:
- C7 pad 2: Net-(U3-PA2) -> Net-(U3-PA0)
- LED1 pad 2: /VBUS -> Net-(LED1-A)
- R4 pad 1: Net-(U3-PA2) -> Net-(U3-PA0)
- U3 pad 10: unconnected-(U3-PA3-Pad10) -> Net-(U3-PA3)
- U3 pad 12: Net-(J3-Pin_1) -> unconnected-(U3-PA5-Pad12)
- U3 pad 13: Net-(J4-Pin_2) -> unconnected-(U3-PA6-Pad13)
- U3 pad 16: unconnected-(U3-PB1-Pad16) -> /D-
- U3 pad 17: unconnected-(U3-PB2-Pad17) -> /D+
- U3 pad 18: unconnected-(U3-PA8-Pad18) -> /SYS_SWDIO
- U3 pad 19: unconnected-(U3-PA9/UCPD1_DBCC1-Pad19) -> /SYS_SWCLK
- U3 pad 7: Net-(Q1-G) -> Net-(U3-PA0)
- U3 pad 8: unconnected-(U3-PA1-Pad8) -> Net-(JP1-A)
- U3 pad 9: Net-(U3-PA2) -> Net-(JP2-A)
Routing:
- net Net-(JP1-A): track 0.00 -> 23.2 mm
- net /D-: track 2.78 -> 22.6 mm
- net /D+: track 2.77 -> 22.5 mm
- net Net-(JP2-A): track 0.00 -> 18.3 mm
- net Net-(U3-PA0): track 0.00 -> 16.8 mm
- net Net-(LED1-A): track 0.00 -> 11.0 mm
- net /3V3: track 30.1 -> 21.1 mm
- net Net-(U3-PA3): track 0.00 -> 8.46 mm, vias 0 -> 2
- net GND: track 19.4 -> 12.6 mm, vias 7 -> 11
- net Net-(J4-Pin_2): track 6.36 -> 0.00 mm
- net /NRST: track 14.7 -> 9.51 mm
- net Net-(Q1-G): track 4.70 -> 0.00 mm
- net Net-(U3-PA2): track 4.49 -> 0.00 mm
- net Net-(J3-Pin_1): track 4.00 -> 0.00 mm
- net /SYS_SWDIO: track 8.05 -> 11.6 mm, vias 2 -> 0
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Other:
- board size 25.2 x 31.2 mm -> 25.2 x 30.2 mm
